File: NAVMAN-GPSBOARD.brd (EAGLE design)
At the start: 90.9 x 72.1 mm, 18 parts, among them X2 SMA-142-0701-801/806

Commit message: Updated gps module design
Routing:
- net GND: track 32.7 -> 26.2 mm, vias 3 -> 2
Changed lines of the file:
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@@
 <text x="57.8" y="57.5" size="1.27" layer="51" font="vector" ratio="12" rot="R90">TXD</text>
 <text x="60.6" y="57.2" size="1.27" layer="51" font="vector" ratio="12" rot="R90">PPSGND</text>
-<text x="63.4" y="57.3" size="1.27" layer="51" font="vector" ratio="12" rot="R90">PPS</text>
+<text x="64.5" y="54.4" size="1.27" layer="51" font="vector" ratio="12" rot="R180">PPS</text>
 <text x="68.5" y="57.2" size="1.27" layer="51" font="vector" ratio="12" rot="R90">10KHZ</text>
 <text x="70.9" y="54.3" size="1.27" layer="51" font="vector" ratio="12" rot="R180">GND</text>
-<text x="74.7" y="54.4" size="1.27" layer="51" font="vector" ratio="12" rot="R180">PWR</text>
+<text x="72.1" y="61.1" size="1.27" layer="51" font="vector" ratio="12" rot="R270">PWR</text>
 <text x="75.1" y="53.2" size="1.27" layer="51" font="vector" ratio="12">BAT</text>
 <text x="2" y="64.1" size="1.27" layer="51" font="vector" ratio="12">+</text>
@@
 <text x="57.6" y="68.9" size="1.27" layer="51" font="vector" ratio="12">V-FTDI</text>
 <text x="42.2" y="68.9" size="1.27" layer="51" font="vector" ratio="12">V-SUPP</text>
+<text x="36.1" y="59.8" size="1.27" layer="51" font="vector" ratio="12">PWR</text>
 </plain>
 <attributes>
@@
 <elements>
 <element name="TU60-D001" library="navman" package="TU60-D001" value="NAVMANJUPITERTU60" x="83.82" y="1.27" rot="R90"/>
-<element name="C1" library="SparkFun-Capacitors" package="CPOL-RADIAL-10UF-25V" value="10uF" x="13.18" y="59.41" rot="R90">
+<element name="C1" library="SparkFun-Capacitors" package="CPOL-RADIAL-10UF-25V" value="10uF" x="13.18" y="59.41" smashed="yes" rot="R90">
 <attribute name="PROD_ID" value="CAP-08440" x="13.18" y="59.41" size="1.778" layer="27" rot="R90" display="off"/>
+<attribute name="NAME" x="12.956" y="56.421" size="1.27" layer="25" font="vector" rot="R180"/>
+<attribute name="VALUE" x="15.263" y="54.705" size="1.27" layer="27" font="vector" rot="R180"/>
 </element>
 <element name="FTDI" library="SparkFun-Connectors" package="1X06_LOCK" value="" x="51.77" y="64.39" smashed="yes">
-<attribute name="NAME" x="51.2" y="65.868" size="1.778" layer="25" font="vector"/>
+<attribute name="NAME" x="57.9" y="65.768" size="1.778" layer="25" font="vector"/>
 <attribute name="VALUE" x="50.5" y="61.088" size="1.27" layer="27" font="vector"/>
 </element>
-<element name="LED1" library="SparkFun-LED" package="LED5MM" value="" x="32.28" y="59.87" rot="R270"/>
+<element name="LED1" library="SparkFun-LED" package="LED5MM" value="" x="32.28" y="59.87" smashed="yes" rot="R270">
+<attribute name="VALUE" x="30.4766" y="56.6696" size="1.27" layer="27" ratio="10" rot="R270"/>
+</element>
 <element name="LED2" library="SparkFun-LED" package="LED5MM" value="" x="76.64" y="60.69" smashed="yes" rot="R180">
 <attribute name="VALUE" x="73.4396" y="62.4934" size="1.27" layer="27" ratio="10" rot="R180"/>
 </element>
-<element name="R1" library="SparkFun-Resistors" package="AXIAL-0.4" value="" x="39.81" y="55.52" rot="R180"/>
-<element name="R2" library="SparkFun-Resistors" package="AXIAL-0.4" value="" x="64.24" y="59.74"/>
+<element name="R1" library="SparkFun-Resistors" package="AXIAL-0.4" value="" x="39.81" y="55.52" smashed="yes" rot="R180">
+<attribute name="NAME" x="40.285" y="58.415" size="1.27" layer="25" font="vector" ratio="15" rot="R180"/>
+<attribute name="VALUE" x="42.096" y="55.901" size="0.8128" layer="21" font="vector" ratio="15" rot="R180"/>
+</element>
+<element name="R2" library="SparkFun-Resistors" package="AXIAL-0.4" value="" x="64.24" y="59.74" smashed="yes">
+<attribute name="NAME" x="63.465" y="61.245" size="1.27" layer="25" font="vector" ratio="15"/>
+<attribute name="VALUE" x="61.954" y="59.359" size="0.8128" layer="21" font="vector" ratio="15"/>
+</element>
 <element name="X1" library="con-wago-500" package="W237-102" value="" x="6.38" y="58.15" rot="R270">
 <attribute name="OC_NEWARK" value="70K9898" x="6.38" y="58.15" size="1.778" layer="27" rot="R270" display="off"/>
@@
 <element name="IC1" library="SparkFun-PowerIC" package="TO220-IGO" value="" x="27.7" y="68.1"/>
 <element name="D2" library="diode" package="DO41-10" value="1N4004" x="22.1" y="61.1"/>
-<element name="JP2" library="SparkFun-Connectors" package="1X03_LOCK" value="" x="50.8" y="69.3"/>
-<element name="C2" library="SparkFun-Capacitors" package="CPOL-RADIAL-10UF-25V" value="10uF" x="19" y="56.1">
+<element name="JP2" library="SparkFun-Connectors" package="1X03_LOCK" value="" x="50.8" y="69.3" smashed="yes">
+<attribute name="NAME" x="51.2538" y="66.4288" size="1.27" layer="25" ratio="10"/>
+<attribute name="VALUE" x="49.53" y="66.125" size="1.27" layer="27"/>
+</element>
+<element name="C2" library="SparkFun-Capacitors" package="CPOL-RADIAL-10UF-25V" value="10uF" x="19" y="56.1" smashed="yes">
 <attribute name="PROD_ID" value="CAP-08440" x="19" y="56.1" size="1.27" layer="27" font="vector" ratio="12" display="off"/>
+<attribute name="NAME" x="22.411" y="56.124" size="1.27" layer="25" font="vector"/>
+<attribute name="VALUE" x="22.495" y="54.517" size="1.27" layer="27" font="vector"/>
 </element>
 </elements>
@@
 </polygon>
 <via x="70.2" y="53.5" extent="1-16" drill="1" shape="square"/>
-<via x="49" y="53.6" extent="1-16" drill="1" shape="square"/>
-<via x="68.2" y="65.4" extent="1-16" drill="1" shape="square"/>
 <contactref element="TP3" pad="TP"/>
 <contactref element="X2" pad="G@1"/>
@@
 <contactref element="X2" pad="G@3"/>
 <contactref element="X2" pad="G@4"/>
-<wire x1="68.2" y1="65.4" x2="72.22" y2="60.38" width="0.6096" layer="1"/>
 <wire x1="72.22" y1="60.38" x2="70.22" y2="55.773" width="0.6096" layer="1"/>
 <wire x1="74.38" y1="41.3" x2="71.4" y2="39.72" width="1.016" layer="1"/>
@@
 </polygon>
 <contactref element="C2" pad="2"/>
-<wire x1="87.5346" y1="33.2196" x2="87.5346" y2="33.2196" width="0" layer="19" extent="1-16"/>
+<via x="88.3" y="37.4" extent="1-16" drill="1" shape="square"/>
 </signal>
 <signal name="VCC">

Commit message: Updated... generated gerbers
Connections:
- removed net PWR: JP1.2
- net VSUP: now also JP1.2
Routing:
- net VSUP: track 66.0 -> 81.0 mm, vias 1 -> 2
- net GND: track 26.2 -> 21.2 mm, vias 2 -> 3
Other:
- board size 90.9 x 72.1 mm -> 90.5 x 72.7 mm
- board text added: "Design by Jason Ball (jason@ball.net)"
- board text added: "GPS Disciplined Oscillator"
- board text added: "Navman Jupiter Tu60"
- board text added: "https://github.com/agronaught/GPS-Disciplined-Oscillator-GPSOXCO-.git"
