File: NAVMAN-GPSBOARD.sch (EAGLE design)
At the start: 18 parts, among them X2 SMA-142-0701-801/806

Commit message: Updated... generated gerbers
Connections:
- removed net PWR: JP1.2
- net VSUP: now also JP1.2
Changed lines of the file:
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@@
-</segment>
-</net>
-<net name="PWR" class="0">
-<segment>
-<pinref part="JP1" gate="G$1" pin="2"/>
-<wire x1="104.14" y1="25.4" x2="109.22" y2="25.4" width="0.1524" layer="91"/>
-<label x="109.22" y="25.4" size="1.27" layer="95" xref="yes"/>
 </segment>
 </net>
@@
 <label x="-5.08" y="50.8" size="1.778" layer="95" rot="R90" xref="yes"/>
 </segment>
+<segment>
+<pinref part="JP1" gate="G$1" pin="2"/>
+<wire x1="104.14" y1="25.4" x2="109.22" y2="25.4" width="0.1524" layer="91"/>
+<label x="109.22" y="25.4" size="1.27" layer="95" xref="yes"/>
+</segment>
 </net>
